Commit message: Old locomotion stack Isaac integration

File: elkapod_description/ros2_control/elkapod.ros2_control.xacro (robot description, xacro)
@@ -1,5 +1,4 @@
 <?xml version="1.0" encoding="utf-8"?>
 <robot xmlns:xacro="http://www.ros.org/wiki/xacro">
-    <!-- Sim mode joint definition -->
     <xacro:macro name="sim_joint_interface" params="name">
         <joint name="${name}">
@@ -12,4 +11,5 @@
     <xacro:macro name="sim_fcp_joint_interface" params="name">
         <joint name="${name}">
+            <command_interface name="position" />
             <state_interface name="position" />
             <state_interface name="velocity" />
@@ -17,5 +17,4 @@
         </joint>
     </xacro:macro>
-    <!-- Real world joint definition -->
     <xacro:macro name="joint_interface" params="name">
         <joint name="${name}">
@@ -24,143 +23,14 @@
         </joint>
     </xacro:macro>
-    <xacro:macro name="elkapod_ros2_control" params="sim_mode:=^|false">
-        <!-- IMU link && joint -->
-        <link name="imu_link" />
-        <joint name="imu_joint" type="fixed">
-            <parent link="base_link" />
-            <child link="imu_link" />
-        </joint>
-        <xacro:if value="${sim_mode}">
-            <!-- Plugins loading -->
-            <gazebo>
-                <plugin name="gz_ros2_control::GazeboSimROS2ControlPlugin"
-                    filename="libgz_ros2_control-system.so">
-                    <parameters>$(find elkapod_description)/config/my_controllers.yaml</parameters>
-                    <!-- <parameters>$(find
-                    elkapod_description)/config/gaz_ros2_ctl_use_sim.yaml</parameters> -->
-                </plugin>
-                <plugin filename="gz-sim-odometry-publisher-system"
-                    name="gz::sim::systems::OdometryPublisher">
-                    <odom_frame>base_link</odom_frame>
-                    <robot_base_frame>base_link</robot_base_frame>
-                    <odom_publish_frequency>50</odom_publish_frequency>
-                    <dimensions>3</dimensions>
-                </plugin>
-            </gazebo>
-            <!-- Joints setup -->
-            <ros2_control name="ElkapodSimHardwareInterface" type="system">
-                <hardware>
-                    <plugin>gz_ros2_control/GazeboSimSystem</plugin>
-                </hardware>
-                <xacro:sim_joint_interface name="leg1_J1" />
-                <xacro:sim_joint_interface name="leg1_J2" />
-                <xacro:sim_joint_interface name="leg1_J3" />
-                <xacro:sim_joint_interface name="leg3_J1" />
-                <xacro:sim_joint_interface name="leg3_J2" />
-                <xacro:sim_joint_interface name="leg3_J3" />
-                <xacro:sim_joint_interface name="leg5_J1" />
-                <xacro:sim_joint_interface name="leg5_J2" />
-                <xacro:sim_joint_interface name="leg5_J3" />
-                <xacro:sim_joint_interface name="leg2_J1" />
-                <xacro:sim_joint_interface name="leg2_J2" />
-                <xacro:sim_joint_interface name="leg2_J3" />
-                <xacro:sim_joint_interface name="leg4_J1" />
-                <xacro:sim_joint_interface name="leg4_J2" />
-                <xacro:sim_joint_interface name="leg4_J3" />
-                <xacro:sim_joint_interface name="leg6_J1" />
-                <xacro:sim_joint_interface name="leg6_J2" />
-                <xacro:sim_joint_interface name="leg6_J3" />
-                <!-- FCP joints (only for joint states broadcaster)-->
-                <xacro:sim_fcp_joint_interface name="leg1_FCP_joint" />
-                <xacro:sim_fcp_joint_interface name="leg2_FCP_joint" />
-                <xacro:sim_fcp_joint_interface name="leg3_FCP_joint" />
-                <xacro:sim_fcp_joint_interface name="leg4_FCP_joint" />
-                <xacro:sim_fcp_joint_interface name="leg5_FCP_joint" />
-                <xacro:sim_fcp_joint_interface name="leg6_FCP_joint" />
-                <!-- Sensors -->
-                <sensor name="imu_sensor" type="imu">
-                    <param name="frame_id">imu_link</param>
-                    <param name="update_rate">50.0</param>
-                    <state_interface name="orientation.x" />
-                    <state_interface name="orientation.y" />
-                    <state_interface name="orientation.z" />
-                    <state_interface name="orientation.w" />
-                    <state_interface name="angular_velocity.x" />
-                    <state_interface name="angular_velocity.y" />
-                    <state_interface name="angular_velocity.z" />
-                    <state_interface name="linear_acceleration.x" />
-                    <state_interface name="linear_acceleration.y" />
-                    <state_interface name="linear_acceleration.z" />
-                </sensor>
-            </ros2_control>
-            <!-- IMU simulation setup -->
-            <gazebo reference="imu_link">
-                <sensor name="imu_sensor" type="imu">
-                    <plugin filename="libgz-sim-imu-system.so" name="gz::sim::systems::Imu">
-                        <initial_orientation_as_reference>false</initial_orientation_as_reference>
-                    </plugin>
-                    <always_on>true</always_on>
-                    <update_rate>100</update_rate>
-                    <visualize>true</visualize>
-                    <imu>
-                        <angular_velocity>
-                            <x>
-                                <noise type="gaussian">
-                                    <mean>0.0</mean>
-                                    <stddev>1e-3</stddev>
-                                    <bias_mean>0.0000075</bias_mean>
-                                    <bias_stddev>0.0000008</bias_stddev>
-                                </noise>
-                            </x>
-                            <y>
-                                <noise type="gaussian">
-                                    <mean>0.0</mean>
-                                    <stddev>1e-3</stddev>
-                                    <bias_mean>0.0000075</bias_mean>
-                                    <bias_stddev>0.0000008</bias_stddev>
-                                </noise>
-                            </y>
-                            <z>
-                                <noise type="gaussian">
-                                    <mean>0.0</mean>
-                                    <stddev>1e-3</stddev>
-                                    <bias_mean>0.0000075</bias_mean>
-                                    <bias_stddev>0.0000008</bias_stddev>
-                                </noise>
-                            </z>
-                        </angular_velocity>
-                        <linear_acceleration>
-                            <x>
-                                <noise type="gaussian">
-                                    <mean>0.0</mean>
-                                    <stddev>1.7e-2</stddev>
-                                    <bias_mean>0.1</bias_mean>
-                                    <bias_stddev>0.001</bias_stddev>
-                                </noise>
-                            </x>
-                            <y>
-                                <noise type="gaussian">
-                                    <mean>0.0</mean>
-                                    <stddev>1.7e-2</stddev>
-                                    <bias_mean>0.1</bias_mean>
-                                    <bias_stddev>0.001</bias_stddev>
-                                </noise>
-                            </y>
-                            <z>
-                                <noise type="gaussian">
-                                    <mean>0.0</mean>
-                                    <stddev>1.7e-2</stddev>
-                                    <bias_mean>0.1</bias_mean>
-                                    <bias_stddev>0.001</bias_stddev>
-                                </noise>
-                            </z>
-                        </linear_acceleration>
-                    </imu>
-                </sensor>
-            </gazebo>
-        </xacro:if>
-        <xacro:unless value="${sim_mode}">
-            <ros2_control name="ElkapodHardwareInterface" type="system">
-                <hardware>
+    <xacro:macro name="elkapod_ros2_control" params="name:='elkapod' sim_mode:=^|false">
+        <ros2_control name="${name}" type="system">
+            <hardware>
+                <xacro:if value="${sim_mode}">
+                    <plugin>topic_based_ros2_control/TopicBasedSystem</plugin>
+                    <param name="joint_commands_topic">/joint_command</param>
+                    <param name="joint_states_topic">/joint_states</param>
+                    <param name="sum_wrapped_joint_states">false</param>
+                </xacro:if>
+                <xacro:unless value="${sim_mode}">
                     <plugin>elkapod_description/elkapod_system_hardware</plugin>
                     <param name="uart_device">/dev/ttyAMA1</param>
@@ -171,40 +41,61 @@
                     <param name="spi_mode">2</param>
                     <param name="spi_speed_hz">1000000</param>
-                </hardware>
+                </xacro:unless>
+            </hardware>
+            <xacro:if value="${sim_mode}">
+                <xacro:sim_joint_interface name="leg1_J1" />
+                <xacro:sim_joint_interface name="leg1_J2" />
+                <xacro:sim_joint_interface name="leg1_J3" />
+                <xacro:sim_joint_interface name="leg2_J1" />
+                <xacro:sim_joint_interface name="leg2_J2" />
+                <xacro:sim_joint_interface name="leg2_J3" />
+                <xacro:sim_joint_interface name="leg3_J1" />
+                <xacro:sim_joint_interface name="leg3_J2" />
+                <xacro:sim_joint_interface name="leg3_J3" />
+                <xacro:sim_joint_interface name="leg4_J1" />
+                <xacro:sim_joint_interface name="leg4_J2" />
+                <xacro:sim_joint_interface name="leg4_J3" />
+                <xacro:sim_joint_interface name="leg5_J1" />
+                <xacro:sim_joint_interface name="leg5_J2" />
+                <xacro:sim_joint_interface name="leg5_J3" />
+                <xacro:sim_joint_interface name="leg6_J1" />
+                <xacro:sim_joint_interface name="leg6_J2" />
+                <xacro:sim_joint_interface name="leg6_J3" />
+                <xacro:sim_fcp_joint_interface name="leg1_FCP_joint" />
+                <xacro:sim_fcp_joint_interface name="leg2_FCP_joint" />
+                <xacro:sim_fcp_joint_interface name="leg3_FCP_joint" />
+                <xacro:sim_fcp_joint_interface name="leg4_FCP_joint" />
+                <xacro:sim_fcp_joint_interface name="leg5_FCP_joint" />
+                <xacro:sim_fcp_joint_interface name="leg6_FCP_joint" />
+            </xacro:if>
+            <xacro:unless value="${sim_mode}">
                 <xacro:joint_interface name="leg1_J1" />
                 <xacro:joint_interface name="leg1_J2" />
                 <xacro:joint_interface name="leg1_J3" />
+                <xacro:joint_interface name="leg2_J1" />
+                <xacro:joint_interface name="leg2_J2" />
+                <xacro:joint_interface name="leg2_J3" />
                 <xacro:joint_interface name="leg3_J1" />
                 <xacro:joint_interface name="leg3_J2" />
                 <xacro:joint_interface name="leg3_J3" />
+                <xacro:joint_interface name="leg4_J1" />
+                <xacro:joint_interface name="leg4_J2" />
+                <xacro:joint_interface name="leg4_J3" />
                 <xacro:joint_interface name="leg5_J1" />
                 <xacro:joint_interface name="leg5_J2" />
                 <xacro:joint_interface name="leg5_J3" />
-                <xacro:joint_interface name="leg2_J1" />
-                <xacro:joint_interface name="leg2_J2" />
-                <xacro:joint_interface name="leg2_J3" />
-                <xacro:joint_interface name="leg4_J1" />
-                <xacro:joint_interface name="leg4_J2" />
-                <xacro:joint_interface name="leg4_J3" />
                 <xacro:joint_interface name="leg6_J1" />
                 <xacro:joint_interface name="leg6_J2" />
                 <xacro:joint_interface name="leg6_J3" />
-                <!-- Sensors -->
-                <sensor name="imu_sensor" type="imu">
-                    <param name="frame_id">imu_link</param>
-                    <param name="update_rate">50.0</param>
-                    <state_interface name="orientation.x" />
-                    <state_interface name="orientation.y" />
-                    <state_interface name="orientation.z" />
-                    <state_interface name="orientation.w" />
-                    <state_interface name="angular_velocity.x" />
-                    <state_interface name="angular_velocity.y" />
-                    <state_interface name="angular_velocity.z" />
-                    <state_interface name="linear_acceleration.x" />
-                    <state_interface name="linear_acceleration.y" />
-                    <state_interface name="linear_acceleration.z" />
-                </sensor>
-            </ros2_control>
-        </xacro:unless>
+            </xacro:unless>
+            <!-- <sensor name="imu_sensor" type="imu">
+                <state_interface name="orientation.x"/><state_interface name="orientation.y"/>
+                <state_interface name="orientation.z"/><state_interface name="orientation.w"/>
+                <state_interface name="angular_velocity.x"/><state_interface name="angular_velocity.y"/>
+                <state_interface name="angular_velocity.z"/>
+                <state_interface name="linear_acceleration.x"/><state_interface name="linear_acceleration.y"/>
+                <state_interface name="linear_acceleration.z"/>
+            </sensor> -->
+        </ros2_control>
     </xacro:macro>
 </robot>

File: elkapod_description/urdf/left_leg/left_leg.urdf.xacro (robot description, xacro)
@@ -163,5 +163,9 @@
     </gazebo>
     <!-- Fixed Joint for FCP -->
+<<<<<<< HEAD
     <joint name="${leg_name}_FCP_joint" type="${fcp_joint_type}">
+=======
+    <joint name="${leg_name}_FCP_joint" type="fixed">
+>>>>>>> 69521bc (Old locomotion stack Isaac integration)
       <origin xyz="0.2135 0.0085747 0" rpy="0 0 -0.29403" />
       <parent link="${leg_name}_linkC" />

File: elkapod_description/urdf/right_leg/right_leg.urdf.xacro (robot description, xacro)
@@ -10,4 +10,6 @@
         <inertia ixx="1.27655E-05" ixy="5.10643E-13" ixz="-2.82428E-08" iyy="2.29991E-05"
           iyz="4.39699E-07" izz="1.62889E-05" />
+        <inertia ixx="1.27655E-05" ixy="5.10643E-13" ixz="-2.82428E-08" iyy="2.29991E-05"
+          iyz="4.39699E-07" izz="1.62889E-05" />
       </inertial>
       <visual>
@@ -16,4 +18,5 @@
           <mesh filename="package://elkapod_description/meshes/right_leg/base_link.STL" />
         </geometry>
+        <material name="leg_black" />
         <material name="leg_black" />
       </visual>
@@ -30,4 +33,8 @@
       <child link="${leg_name}_base_link" />
       <axis xyz="0 0 0" />
+      <origin xyz="${pos_x} ${pos_y} ${pos_z}" rpy="${roll} ${pitch} ${yaw}" />
+      <parent link="${parent}" />
+      <child link="${leg_name}_base_link" />
+      <axis xyz="0 0 0" />
     </joint>
     <!-- Link A -->
@@ -38,4 +45,6 @@
         <inertia ixx="1.98022E-05" ixy="-2.13458E-13" ixz="-5.41372E-13" iyy="1.670609E-05"
           iyz="-2.17248E-12" izz="1.67061E-05" />
+        <inertia ixx="1.98022E-05" ixy="-2.13458E-13" ixz="-5.41372E-13" iyy="1.670609E-05"
+          iyz="-2.17248E-12" izz="1.67061E-05" />
       </inertial>
       <visual>
@@ -44,4 +53,5 @@
           <mesh filename="package://elkapod_description/meshes/right_leg/linkA.STL" />
         </geometry>
+        <material name="leg_black" />
         <material name="leg_black" />
       </visual>
@@ -68,4 +78,6 @@
         <inertia ixx="2.79458E-05" ixy="8.13719E-13" ixz="2.16502E-12" iyy="4.53975E-05"
           iyz="-7.11437E-07" izz="3.38637E-05" />
+        <inertia ixx="2.79458E-05" ixy="8.13719E-13" ixz="2.16502E-12" iyy="4.53975E-05"
+          iyz="-7.11437E-07" izz="3.38637E-05" />
       </inertial>
       <visual>
@@ -74,4 +86,5 @@
           <mesh filename="package://elkapod_description/meshes/right_leg/linkB.STL" />
         </geometry>
+        <material name="leg_black" />
         <material name="leg_black" />
       </visual>
@@ -98,4 +111,6 @@
         <inertia ixx="1.77293E-05" ixy="-3.34917E-06" ixz="3.26962E-07" iyy="6.16756E-05"
           iyz="6.79304E-08" izz="5.23429E-05" />
+        <inertia ixx="1.77293E-05" ixy="-3.34917E-06" ixz="3.26962E-07" iyy="6.16756E-05"
+          iyz="6.79304E-08" izz="5.23429E-05" />
       </inertial>
       <visual>
@@ -104,4 +119,5 @@
           <mesh filename="package://elkapod_description/meshes/right_leg/linkC.STL" />
         </geometry>
+        <material name="orange_pla" />
         <material name="orange_pla" />
       </visual>
@@ -128,8 +144,11 @@
         <inertia ixx="1.19862E-06" ixy="1.05879E-22" ixz="1.15499E-24" iyy="1.06703E-06"
           iyz="9.44775E-26" izz="1.06703E-06" />
+        <inertia ixx="1.19862E-06" ixy="1.05879E-22" ixz="1.15499E-24" iyy="1.06703E-06"
+          iyz="9.44775E-26" izz="1.06703E-06" />
       </inertial>
       <visual>
         <origin xyz="0 0 0" rpy="0 0 0" />
         <geometry>
+          <sphere radius="0.01" />
           <sphere radius="0.01" />
         </geometry>
@@ -141,4 +160,5 @@
         <origin xyz="0 0 0" rpy="0 0 0" />
         <geometry>
+          <sphere radius="0.01" />
           <sphere radius="0.01" />
         </geometry>
