Commit message: Fix joint limits precision, format, add fcp_joint_type parameter to URDF

File: elkapod_description/ros2_control/elkapod.ros2_control.xacro (robot description, xacro)
@@ -4,15 +4,15 @@
     <xacro:macro name="sim_joint_interface" params="name">
         <joint name="${name}">
-            <command_interface name="position"/>
-            <state_interface name="position"/>
-            <state_interface name="velocity"/>
-            <state_interface name="effort"/>
+            <command_interface name="position" />
+            <state_interface name="position" />
+            <state_interface name="velocity" />
+            <state_interface name="effort" />
         </joint>
     </xacro:macro>
     <xacro:macro name="sim_fcp_joint_interface" params="name">
         <joint name="${name}">
-            <state_interface name="position"/>
-            <state_interface name="velocity"/>
-            <state_interface name="effort"/>
+            <state_interface name="position" />
+            <state_interface name="velocity" />
+            <state_interface name="effort" />
         </joint>
     </xacro:macro>
@@ -20,23 +20,26 @@
     <xacro:macro name="joint_interface" params="name">
         <joint name="${name}">
-            <command_interface name="position"/>
-            <state_interface name="position"/>
+            <command_interface name="position" />
+            <state_interface name="position" />
         </joint>
     </xacro:macro>
     <xacro:macro name="elkapod_ros2_control" params="sim_mode:=^|false">
         <!-- IMU link && joint -->
-        <link name="imu_link"/>
+        <link name="imu_link" />
         <joint name="imu_joint" type="fixed">
-            <parent link="base_link"/>
-            <child link="imu_link"/>
+            <parent link="base_link" />
+            <child link="imu_link" />
         </joint>
         <xacro:if value="${sim_mode}">
             <!-- Plugins loading -->
             <gazebo>
-                <plugin name="gz_ros2_control::GazeboSimROS2ControlPlugin" filename="libgz_ros2_control-system.so">
+                <plugin name="gz_ros2_control::GazeboSimROS2ControlPlugin"
+                    filename="libgz_ros2_control-system.so">
                     <parameters>$(find elkapod_description)/config/my_controllers.yaml</parameters>
-                    <!-- <parameters>$(find elkapod_description)/config/gaz_ros2_ctl_use_sim.yaml</parameters> -->
+                    <!-- <parameters>$(find
+                    elkapod_description)/config/gaz_ros2_ctl_use_sim.yaml</parameters> -->
                 </plugin>
-                <plugin filename="gz-sim-odometry-publisher-system" name="gz::sim::systems::OdometryPublisher">
+                <plugin filename="gz-sim-odometry-publisher-system"
+                    name="gz::sim::systems::OdometryPublisher">
                     <odom_frame>base_link</odom_frame>
                     <robot_base_frame>base_link</robot_base_frame>
@@ -50,43 +53,43 @@
                     <plugin>gz_ros2_control/GazeboSimSystem</plugin>
                 </hardware>
-                <xacro:sim_joint_interface name="leg1_J1"/>
-                <xacro:sim_joint_interface name="leg1_J2"/>
-                <xacro:sim_joint_interface name="leg1_J3"/>
-                <xacro:sim_joint_interface name="leg3_J1"/>
-                <xacro:sim_joint_interface name="leg3_J2"/>
-                <xacro:sim_joint_interface name="leg3_J3"/>
-                <xacro:sim_joint_interface name="leg5_J1"/>
-                <xacro:sim_joint_interface name="leg5_J2"/>
-                <xacro:sim_joint_interface name="leg5_J3"/>
-                <xacro:sim_joint_interface name="leg2_J1"/>
-                <xacro:sim_joint_interface name="leg2_J2"/>
-                <xacro:sim_joint_interface name="leg2_J3"/>
-                <xacro:sim_joint_interface name="leg4_J1"/>
-                <xacro:sim_joint_interface name="leg4_J2"/>
-                <xacro:sim_joint_interface name="leg4_J3"/>
-                <xacro:sim_joint_interface name="leg6_J1"/>
-                <xacro:sim_joint_interface name="leg6_J2"/>
-                <xacro:sim_joint_interface name="leg6_J3"/>
+                <xacro:sim_joint_interface name="leg1_J1" />
+                <xacro:sim_joint_interface name="leg1_J2" />
+                <xacro:sim_joint_interface name="leg1_J3" />
+                <xacro:sim_joint_interface name="leg3_J1" />
+                <xacro:sim_joint_interface name="leg3_J2" />
+                <xacro:sim_joint_interface name="leg3_J3" />
+                <xacro:sim_joint_interface name="leg5_J1" />
+                <xacro:sim_joint_interface name="leg5_J2" />
+                <xacro:sim_joint_interface name="leg5_J3" />
+                <xacro:sim_joint_interface name="leg2_J1" />
+                <xacro:sim_joint_interface name="leg2_J2" />
+                <xacro:sim_joint_interface name="leg2_J3" />
+                <xacro:sim_joint_interface name="leg4_J1" />
+                <xacro:sim_joint_interface name="leg4_J2" />
+                <xacro:sim_joint_interface name="leg4_J3" />
+                <xacro:sim_joint_interface name="leg6_J1" />
+                <xacro:sim_joint_interface name="leg6_J2" />
+                <xacro:sim_joint_interface name="leg6_J3" />
                 <!-- FCP joints (only for joint states broadcaster)-->
-                <xacro:sim_fcp_joint_interface name="leg1_FCP_joint"/>
-                <xacro:sim_fcp_joint_interface name="leg2_FCP_joint"/>
-                <xacro:sim_fcp_joint_interface name="leg3_FCP_joint"/>
-                <xacro:sim_fcp_joint_interface name="leg4_FCP_joint"/>
-                <xacro:sim_fcp_joint_interface name="leg5_FCP_joint"/>
-                <xacro:sim_fcp_joint_interface name="leg6_FCP_joint"/>
+                <xacro:sim_fcp_joint_interface name="leg1_FCP_joint" />
+                <xacro:sim_fcp_joint_interface name="leg2_FCP_joint" />
+                <xacro:sim_fcp_joint_interface name="leg3_FCP_joint" />
+                <xacro:sim_fcp_joint_interface name="leg4_FCP_joint" />
+                <xacro:sim_fcp_joint_interface name="leg5_FCP_joint" />
+                <xacro:sim_fcp_joint_interface name="leg6_FCP_joint" />
                 <!-- Sensors -->
                 <sensor name="imu_sensor" type="imu">
                     <param name="frame_id">imu_link</param>
                     <param name="update_rate">50.0</param>
-                    <state_interface name="orientation.x"/>
-                    <state_interface name="orientation.y"/>
-                    <state_interface name="orientation.z"/>
-                    <state_interface name="orientation.w"/>
-                    <state_interface name="angular_velocity.x"/>
-                    <state_interface name="angular_velocity.y"/>
-                    <state_interface name="angular_velocity.z"/>
-                    <state_interface name="linear_acceleration.x"/>
-                    <state_interface name="linear_acceleration.y"/>
-                    <state_interface name="linear_acceleration.z"/>
+                    <state_interface name="orientation.x" />
+                    <state_interface name="orientation.y" />
+                    <state_interface name="orientation.z" />
+                    <state_interface name="orientation.w" />
+                    <state_interface name="angular_velocity.x" />
+                    <state_interface name="angular_velocity.y" />
+                    <state_interface name="angular_velocity.z" />
+                    <state_interface name="linear_acceleration.x" />
+                    <state_interface name="linear_acceleration.y" />
+                    <state_interface name="linear_acceleration.z" />
                 </sensor>
             </ros2_control>
@@ -169,36 +172,36 @@
                     <param name="spi_speed_hz">1000000</param>
                 </hardware>
-                <xacro:joint_interface name="leg1_J1"/>
-                <xacro:joint_interface name="leg1_J2"/>
-                <xacro:joint_interface name="leg1_J3"/>
-                <xacro:joint_interface name="leg3_J1"/>
-                <xacro:joint_interface name="leg3_J2"/>
-                <xacro:joint_interface name="leg3_J3"/>
-                <xacro:joint_interface name="leg5_J1"/>
-                <xacro:joint_interface name="leg5_J2"/>
-                <xacro:joint_interface name="leg5_J3"/>
-                <xacro:joint_interface name="leg2_J1"/>
-                <xacro:joint_interface name="leg2_J2"/>
-                <xacro:joint_interface name="leg2_J3"/>
-                <xacro:joint_interface name="leg4_J1"/>
-                <xacro:joint_interface name="leg4_J2"/>
-                <xacro:joint_interface name="leg4_J3"/>
-                <xacro:joint_interface name="leg6_J1"/>
-                <xacro:joint_interface name="leg6_J2"/>
-                <xacro:joint_interface name="leg6_J3"/>
+                <xacro:joint_interface name="leg1_J1" />
+                <xacro:joint_interface name="leg1_J2" />
+                <xacro:joint_interface name="leg1_J3" />
+                <xacro:joint_interface name="leg3_J1" />
+                <xacro:joint_interface name="leg3_J2" />
+                <xacro:joint_interface name="leg3_J3" />
+                <xacro:joint_interface name="leg5_J1" />
+                <xacro:joint_interface name="leg5_J2" />
+                <xacro:joint_interface name="leg5_J3" />
+                <xacro:joint_interface name="leg2_J1" />
+                <xacro:joint_interface name="leg2_J2" />
+                <xacro:joint_interface name="leg2_J3" />
+                <xacro:joint_interface name="leg4_J1" />
+                <xacro:joint_interface name="leg4_J2" />
+                <xacro:joint_interface name="leg4_J3" />
+                <xacro:joint_interface name="leg6_J1" />
+                <xacro:joint_interface name="leg6_J2" />
+                <xacro:joint_interface name="leg6_J3" />
                 <!-- Sensors -->
                 <sensor name="imu_sensor" type="imu">
                     <param name="frame_id">imu_link</param>
                     <param name="update_rate">50.0</param>
-                    <state_interface name="orientation.x"/>
-                    <state_interface name="orientation.y"/>
-                    <state_interface name="orientation.z"/>
-                    <state_interface name="orientation.w"/>
-                    <state_interface name="angular_velocity.x"/>
-                    <state_interface name="angular_velocity.y"/>
-                    <state_interface name="angular_velocity.z"/>
-                    <state_interface name="linear_acceleration.x"/>
-                    <state_interface name="linear_acceleration.y"/>
-                    <state_interface name="linear_acceleration.z"/>
+                    <state_interface name="orientation.x" />
+                    <state_interface name="orientation.y" />
+                    <state_interface name="orientation.z" />
+                    <state_interface name="orientation.w" />
+                    <state_interface name="angular_velocity.x" />
+                    <state_interface name="angular_velocity.y" />
+                    <state_interface name="angular_velocity.z" />
+                    <state_interface name="linear_acceleration.x" />
+                    <state_interface name="linear_acceleration.y" />
+                    <state_interface name="linear_acceleration.z" />
                 </sensor>
             </ros2_control>

File: elkapod_description/urdf/body/body.urdf.xacro (robot description, xacro)
@@ -1,9 +1,9 @@
 <?xml version="1.0" encoding="utf-8"?>
 <robot xmlns:xacro="http://ros.org/wiki/xacro">
-  <link name="base_link"/>
+  <link name="base_link" />
   <joint name="base_body_link" type="fixed">
-        <parent link="base_link"/>
-        <child link="body_link"/>
-        <origin xyz="0 0 0" rpy="0 0 0"/>
+    <parent link="base_link" />
+    <child link="body_link" />
+    <origin xyz="0 0 0" rpy="0 0 0" />
   </joint>
   <link name="body_link">
@@ -13,5 +13,6 @@
         rpy="0 0 0" />
       <mass value="2.0043" />
-      <inertia ixx="0.0094039" ixy="0.00013899" ixz="-4.7517E-07" iyy="0.014031" iyz="1.9401E-09" izz="0.023053" />
+      <inertia ixx="0.0094039" ixy="0.00013899" ixz="-4.7517E-07" iyy="0.014031" iyz="1.9401E-09"
+        izz="0.023053" />
     </inertial>
     <visual>
@@ -20,5 +21,5 @@
         <mesh filename="package://elkapod_description/meshes/body/base_link.STL" />
       </geometry>
-      <material name="aluminium_base"/>
+      <material name="aluminium_base" />
     </visual>
     <collision>
@@ -33,5 +34,6 @@
       <origin xyz="0.004012 0.03538 -0.0033877" rpy="0 0 0" />
       <mass value="0.43861" />
-      <inertia ixx="0.00085006" ixy="-1.6091E-05" ixz="-1.9773E-06" iyy="0.0021513" iyz="1.4281E-05" izz="0.0014553" />
+      <inertia ixx="0.00085006" ixy="-1.6091E-05" ixz="-1.9773E-06" iyy="0.0021513" iyz="1.4281E-05"
+        izz="0.0014553" />
     </inertial>
     <visual>
@@ -40,5 +42,5 @@
         <mesh filename="package://elkapod_description/meshes/body/control_module.STL" />
       </geometry>
-      <material name="orange_pla"/>
+      <material name="orange_pla" />
     </visual>
     <collision>
@@ -59,5 +61,6 @@
       <origin xyz="-1.2221E-17 0.00073241 -0.0031202" rpy="0 0 0" />
       <mass value="0.051567" />
-      <inertia ixx="2.0691E-05" ixy="-6.8955E-21" ixz="-3.4656E-20" iyy="0.00017525" iyz="4.3338E-07" izz="0.00019204" />
+      <inertia ixx="2.0691E-05" ixy="-6.8955E-21" ixz="-3.4656E-20" iyy="0.00017525"
+        iyz="4.3338E-07" izz="0.00019204" />
     </inertial>
     <visual>
@@ -66,5 +69,5 @@
         <mesh filename="package://elkapod_description/meshes/body/front_grille.STL" />
       </geometry>
-      <material name="orange_pla"/>
+      <material name="orange_pla" />
     </visual>
     <collision>
@@ -76,5 +79,5 @@
   </link>
   <joint name="front_grille_fixed" type="fixed">
-    <origin xyz="0.1623 0 0" rpy="1.5708 0 1.5708" />
+    <origin xyz="0.1623 0 0" rpy="1.570796327 0 1.570796327" />
     <parent link="base_link" />
     <child link="front_grille" />
@@ -85,5 +88,6 @@
       <origin xyz="0.058453 0.03 0.0029846" rpy="0 0 0" />
       <mass value="0.042927" />
-      <inertia ixx="1.6075E-05" ixy="1.7888E-19" ixz="1.0449E-08" iyy="1.0788E-05" iyz="4.1841E-20" izz="2.593E-05" />
+      <inertia ixx="1.6075E-05" ixy="1.7888E-19" ixz="1.0449E-08" iyy="1.0788E-05" iyz="4.1841E-20"
+        izz="2.593E-05" />
     </inertial>
     <visual>
@@ -92,5 +96,5 @@
         <mesh filename="package://elkapod_description/meshes/body/back_grilles.STL" />
       </geometry>
-      <material name="orange_pla"/>
+      <material name="orange_pla" />
     </visual>
     <collision>
@@ -102,5 +106,5 @@
   </link>
   <joint name="back_grilles_fixed" type="fixed">
-    <origin xyz="-0.15412 0.059195 -0.03" rpy="1.5708 0 -1.5708" />
+    <origin xyz="-0.15412 0.059195 -0.03" rpy="1.570796327 0 -1.570796327" />
     <parent link="base_link" />
     <child link="back_grilles" />
@@ -111,5 +115,6 @@
       <origin xyz="0.07377 0.03 -0.037189" rpy="0 0 0" />
       <mass value="0.016676" />
-      <inertia ixx="1.8158E-05" ixy="4.5854E-21" ixz="-2.8456E-19" iyy="1.1749E-05" iyz="3.0718E-12" izz="6.6615E-06" />
+      <inertia ixx="1.8158E-05" ixy="4.5854E-21" ixz="-2.8456E-19" iyy="1.1749E-05" iyz="3.0718E-12"
+        izz="6.6615E-06" />
     </inertial>
     <visual>
@@ -118,5 +123,5 @@
         <mesh filename="package://elkapod_description/meshes/body/left_side_grille.STL" />
       </geometry>
-      <material name="black_pla"/>
+      <material name="black_pla" />
     </visual>
     <collision>
@@ -128,5 +133,5 @@
   </link>
   <joint name="left_side_grille_fixed" type="fixed">
-    <origin xyz="0.039489 0.19711 0.03" rpy="-1.5708 0 -1.5708" />
+    <origin xyz="0.039489 0.19711 0.03" rpy="-1.570796327 0 -1.570796327" />
     <parent link="base_link" />
     <child link="left_side_grille" />
@@ -140,5 +145,6 @@
       <mass
         value="0.016676" />
-      <inertia ixx="1.8158E-05" ixy="-4.8096E-22" ixz="1.1647E-21" iyy="1.1749E-05" iyz="3.0718E-12" izz="6.6615E-06" />
+      <inertia ixx="1.8158E-05" ixy="-4.8096E-22" ixz="1.1647E-21" iyy="1.1749E-05" iyz="3.0718E-12"
+        izz="6.6615E-06" />
     </inertial>
     <visual>
@@ -147,5 +153,5 @@
         <mesh filename="package://elkapod_description/meshes/body/right_side_grille.STL" />
       </geometry>
-      <material name="black_pla"/>
+      <material name="black_pla" />
     </visual>
     <collision>
@@ -157,5 +163,5 @@
   </link>
   <joint name="right_side_grille_fixed" type="fixed">
-    <origin xyz="-0.034889 -0.19711 0.03" rpy="-1.5708 0 1.5708" />
+    <origin xyz="-0.034889 -0.19711 0.03" rpy="-1.570796327 0 1.570796327" />
     <parent link="base_link" />
     <child link="right_side_grille" />
@@ -175,5 +181,5 @@
         <mesh filename="package://elkapod_description/meshes/body/rubber_feet.STL" />
       </geometry>
-      <material name="pure_black"/>
+      <material name="pure_black" />
     </visual>
     <collision>

File: elkapod_description/urdf/colors.urdf.xacro (robot description, xacro)
@@ -2,21 +2,21 @@
 <robot xmlns:xacro="http://www.ros.org/wiki/xacro">
     <material name="orange_pla">
-        <color rgba="0.9411 0.4196 0.0470 1"/>
+        <color rgba="0.9411 0.4196 0.0470 1" />
     </material>
     <material name="pure_black">
-        <color rgba="0 0 0 1"/>
+        <color rgba="0 0 0 1" />
     </material>
     <material name="lidar_black">
-        <color rgba="0.025 0.025 0.025 1"/>
+        <color rgba="0.025 0.025 0.025 1" />
         <specular>1.0 1.0 1.0 1.0</specular>
     </material>
     <material name="black_pla">
-        <color rgba="0.05 0.05 0.05 1"/>
+        <color rgba="0.05 0.05 0.05 1" />
     </material>
     <material name="leg_black">
-        <color rgba="0.25098 0.25098 0.25098 1"/>
+        <color rgba="0.25098 0.25098 0.25098 1" />
     </material>
     <material name="aluminium_base">
-        <color rgba="0.8902 0.8902 0.91373 1"/>
+        <color rgba="0.8902 0.8902 0.91373 1" />
     </material>
 </robot>

File: elkapod_description/urdf/elkapod.urdf.xacro (robot description, xacro)
@@ -2,5 +2,5 @@
 <robot xmlns:xacro="http://ros.org/wiki/xacro" name="elkapod">
   <!-- Execution env config -->
-  <xacro:arg name="sim_mode" default="false"/>
+  <xacro:arg name="sim_mode" default="false" />
   <!-- INCLUDES -->
   <!-- Colors -->
@@ -9,19 +9,27 @@
   <xacro:include filename="$(find elkapod_description)/urdf/body/body.urdf.xacro" />
   <!-- Legs-->
+  <xacro:arg name="fcp_joint_type" default="prismatic" />
   <xacro:include filename="$(find elkapod_description)/urdf/left_leg/left_leg.urdf.xacro" />
   <xacro:include filename="$(find elkapod_description)/urdf/right_leg/right_leg.urdf.xacro" />
-  <xacro:leg_left leg_name="leg1" parent="base_link" pos_x="0.17841" pos_y="0.13276" pos_z="-0.03" roll="0" pitch="0" yaw="0.63973287"/>
-  <xacro:leg_left leg_name="leg3" parent="base_link" pos_x="0.0138" pos_y="0.1643" pos_z="-0.03" roll="0" pitch="0" yaw="1.57"/>
-  <xacro:leg_left leg_name="leg5" parent="base_link" pos_x="-0.15903" pos_y="0.15038" pos_z="-0.03" roll="0" pitch="0" yaw="2.384143643587"/>
-  <xacro:leg_right leg_name="leg2" parent="base_link" pos_x="0.17841" pos_y="-0.13276" pos_z="-0.03" roll="0" pitch="0" yaw="-0.63973287"/>
-  <xacro:leg_right leg_name="leg4" parent="base_link" pos_x="0.0138" pos_y="-0.1643" pos_z="-0.03" roll="0" pitch="0" yaw="-1.57"/>
-  <xacro:leg_right leg_name="leg6" parent="base_link" pos_x="-0.15903" pos_y="-0.15038" pos_z="-0.03" roll="0" pitch="0" yaw="-2.384143643587"/>
+  <xacro:leg_left leg_name="leg1" parent="base_link" pos_x="0.17841" pos_y="0.13276" pos_z="-0.03"
+    roll="0" pitch="0" yaw="0.63973287" fcp_joint_type="$(arg fcp_joint_type)" />
+  <xacro:leg_left leg_name="leg3" parent="base_link" pos_x="0.0138" pos_y="0.1643" pos_z="-0.03"
+    roll="0" pitch="0" yaw="1.570796327" fcp_joint_type="$(arg fcp_joint_type)" />
+  <xacro:leg_left leg_name="leg5" parent="base_link" pos_x="-0.15903" pos_y="0.15038" pos_z="-0.03"
+    roll="0" pitch="0" yaw="2.384143643587" fcp_joint_type="$(arg fcp_joint_type)" />
+  <xacro:leg_right leg_name="leg2" parent="base_link" pos_x="0.17841" pos_y="-0.13276" pos_z="-0.03"
+    roll="0" pitch="0" yaw="-0.63973287" fcp_joint_type="$(arg fcp_joint_type)" />
+  <xacro:leg_right leg_name="leg4" parent="base_link" pos_x="0.0138" pos_y="-0.1643" pos_z="-0.03"
+    roll="0" pitch="0" yaw="-1.570796327" fcp_joint_type="$(arg fcp_joint_type)" />
+  <xacro:leg_right leg_name="leg6" parent="base_link" pos_x="-0.15903" pos_y="-0.15038"
+    pos_z="-0.03" roll="0" pitch="0" yaw="-2.384143643587" fcp_joint_type="$(arg fcp_joint_type)" />
   <!-- Sensors -->
   <xacro:include filename="$(find elkapod_description)/urdf/sensors/lidar.xacro" />
   <xacro:include filename="$(find elkapod_description)/urdf/sensors/depth_camera.xacro" />
-  <xacro:elkapod_sensors_lidar sim_mode="$(arg sim_mode)"/>
-  <xacro:elkapod_sensors_fron_camera sim_mode="$(arg sim_mode)"/>
+  <xacro:elkapod_sensors_lidar sim_mode="$(arg sim_mode)" />
+  <!-- Fixed potential typo from 'fron_camera' to 'front_camera' -->
+  <xacro:elkapod_sensors_front_camera sim_mode="$(arg sim_mode)" />
   <!-- ros2_control -->
   <xacro:include filename="$(find elkapod_description)/ros2_control/elkapod.ros2_control.xacro" />
-  <xacro:elkapod_ros2_control sim_mode="$(arg sim_mode)"/>
+  <xacro:elkapod_ros2_control sim_mode="$(arg sim_mode)" />
 </robot>
