Commit message: Fix joint limits precision, format, add fcp_joint_type parameter to URDF

File: elkapod_description/urdf/left_leg/left_leg.urdf.xacro (robot description, xacro)
@@ -1,5 +1,6 @@
 <?xml version="1.0" encoding="utf-8"?>
 <robot xmlns:xacro="http://ros.org/wiki/xacro">
-  <xacro:macro name="leg_left" params="leg_name parent pos_x pos_y pos_z roll pitch yaw">
+  <xacro:macro name="leg_left"
+    params="leg_name parent pos_x pos_y pos_z roll pitch yaw fcp_joint_type:=prismatic">
     <!-- Base Link -->
     <link name="${leg_name}_base_link">
@@ -7,5 +8,6 @@
         <origin xyz="-0.0097901 0.0013901 0.021894" rpy="0 0 0" />
         <mass value="0.080802" />
-        <inertia ixx="1.2766E-05" ixy="5.3087E-13" ixz="-2.8241E-08" iyy="2.2999E-05" iyz="-4.397E-07" izz="1.6289E-05" />
+        <inertia ixx="1.2766E-05" ixy="5.3087E-13" ixz="-2.8241E-08" iyy="2.2999E-05"
+          iyz="-4.397E-07" izz="1.6289E-05" />
       </inertial>
       <visual>
@@ -14,5 +16,5 @@
           <mesh filename="package://elkapod_description/meshes/left_leg/base_link.STL" />
         </geometry>
-        <material name="leg_black"/>
+        <material name="leg_black" />
       </visual>
       <collision>
@@ -34,5 +36,6 @@
         <origin xyz="0.033799 0.00051236 0.00054959" rpy="0 0 0" />
         <mass value="0.042693" />
-        <inertia ixx="1.9802E-05" ixy="8.7559E-13" ixz="-5.8218E-13" iyy="1.6706E-05" iyz="-1.8291E-12" izz="1.6706E-05" />
+        <inertia ixx="1.9802E-05" ixy="8.7559E-13" ixz="-5.8218E-13" iyy="1.6706E-05"
+          iyz="-1.8291E-12" izz="1.6706E-05" />
       </inertial>
       <visual>
@@ -41,5 +44,5 @@
           <mesh filename="package://elkapod_description/meshes/left_leg/linkA.STL" />
         </geometry>
-        <material name="leg_black"/>
+        <material name="leg_black" />
       </visual>
       <collision>
@@ -56,5 +59,5 @@
       <child link="${leg_name}_linkA" />
       <axis xyz="0 0 1" />
-      <limit lower="-1.57" upper="1.57" effort="50.0" velocity="7.3" />
+      <limit lower="-1.570796327" upper="1.570796327" effort="50.0" velocity="7.3" />
     </joint>
     <!-- Link B -->
@@ -63,5 +66,6 @@
         <origin xyz="0.046185 0.0047076 0.0034661" rpy="0 0 0" />
         <mass value="0.16871" />
-        <inertia ixx="2.7946E-05" ixy="-8.4625E-13" ixz="2.1218E-12" iyy="4.5398E-05" iyz="7.1144E-07" izz="3.3864E-05" />
+        <inertia ixx="2.7946E-05" ixy="-8.4625E-13" ixz="2.1218E-12" iyy="4.5398E-05"
+          iyz="7.1144E-07" izz="3.3864E-05" />
       </inertial>
       <visual>
@@ -70,5 +74,5 @@
           <mesh filename="package://elkapod_description/meshes/left_leg/linkB.STL" />
         </geometry>
-        <material name="leg_black"/>
+        <material name="leg_black" />
       </visual>
       <collision>
@@ -81,9 +85,9 @@
     <!-- Joint J2 -->
     <joint name="${leg_name}_J2" type="revolute">
-      <origin xyz="0.0676 0 0" rpy="1.5708 0 0" />
+      <origin xyz="0.0676 0 0" rpy="1.570796327 0 0" />
       <parent link="${leg_name}_linkA" />
       <child link="${leg_name}_linkB" />
       <axis xyz="0 0 1" />
-      <limit lower="-1.57" upper="1.57" effort="50.0" velocity="7.3" />
+      <limit lower="-1.570796327" upper="1.570796327" effort="50.0" velocity="7.3" />
     </joint>
     <!-- Link C -->
@@ -92,5 +96,6 @@
         <origin xyz="0.062526 0.013836 -0.00039598" rpy="0 0 0" />
         <mass value="0.045919" />
-        <inertia ixx="1.7731E-05" ixy="-3.3492E-06" ixz="3.2696E-07" iyy="6.1677E-05" iyz="6.793E-08" izz="5.2343E-05" />
+        <inertia ixx="1.7731E-05" ixy="-3.3492E-06" ixz="3.2696E-07" iyy="6.1677E-05"
+          iyz="6.793E-08" izz="5.2343E-05" />
       </inertial>
       <visual>
@@ -99,5 +104,5 @@
           <mesh filename="package://elkapod_description/meshes/left_leg/linkC.STL" />
         </geometry>
-        <material name="orange_pla"/>
+        <material name="orange_pla" />
       </visual>
       <collision>
@@ -114,5 +119,5 @@
       <child link="${leg_name}_linkC" />
       <axis xyz="0 0 1" />
-      <limit lower="-3.14" upper="1.57" effort="50.0" velocity="7.3" />
+      <limit lower="-3.141592654" upper="0.0" effort="50.0" velocity="7.3" />
     </joint>
     <!-- FCP Link -->
@@ -121,10 +126,11 @@
         <origin xyz="0.000341547110339208 2.77555756156289E-17 1.73472347597681E-18" rpy="0 0 0" />
         <mass value="0.0111617991818567" />
-        <inertia ixx="1.19862E-06" ixy="-5.67881E-40" ixz="-4.86711E-24" iyy="1.06703E-06" iyz="-1.94856E-26" izz="1.06703E-06" />
+        <inertia ixx="1.19862E-06" ixy="-5.67881E-40" ixz="-4.86711E-24" iyy="1.06703E-06"
+          iyz="-1.94856E-26" izz="1.06703E-06" />
       </inertial>
       <visual>
         <origin xyz="0 0 0" rpy="0 0 0" />
         <geometry>
-          <sphere radius="0.01"/>
+          <sphere radius="0.01" />
         </geometry>
         <material name="">
@@ -135,5 +141,5 @@
         <origin xyz="0 0 0" rpy="0 0 0" />
         <geometry>
-          <sphere radius="0.01"/>
+          <sphere radius="0.01" />
         </geometry>
       </collision>
@@ -146,18 +152,4 @@
       <minDepth>0.01</minDepth>
     </gazebo>
-    <!-- <gazebo reference="${leg_name}_FCP_joint">
-        <sensor name="${leg_name}_fsr" type="force_torque">
-          <always_on>true</always_on>
-          <update_rate>100</update_rate>
-          <visualize>true</visualize>
-          <topic>/legs/${leg_name}_fsr</topic>
-          <enable_metrics>true</enable_metrics>
-          <pose>0 0 0 0 0 0</pose>
-          <force_torque>
-            <frame>sensor</frame>
-            <measure_direction>child_to_parent</measure_direction>
-          </force_torque>
-        </sensor>
-    </gazebo> -->
     <gazebo reference="${leg_name}_FCP">
       <sensor name="contact" type="contact">
@@ -171,11 +163,11 @@
     </gazebo>
     <!-- Fixed Joint for FCP -->
-    <joint name="${leg_name}_FCP_joint" type="prismatic">
+    <joint name="${leg_name}_FCP_joint" type="${fcp_joint_type}">
       <origin xyz="0.2135 0.0085747 0" rpy="0 0 -0.29403" />
       <parent link="${leg_name}_linkC" />
       <child link="${leg_name}_FCP" />
       <axis xyz="1 0 0" />
-      <limit effort="1000.0" lower="-0.0001" upper="0.0001" velocity="30"/>
-      <dynamics damping="10.0" friction="0.0"/>
+      <limit effort="1000.0" lower="-0.0001" upper="0.0001" velocity="30" />
+      <dynamics damping="10.0" friction="0.0" />
     </joint>
   </xacro:macro>

File: elkapod_description/urdf/right_leg/right_leg.urdf.xacro (robot description, xacro)
@@ -1,5 +1,6 @@
 <?xml version="1.0" encoding="utf-8"?>
 <robot xmlns:xacro="http://ros.org/wiki/xacro">
-  <xacro:macro name="leg_right" params="leg_name parent pos_x pos_y pos_z roll pitch yaw">
+  <xacro:macro name="leg_right"
+    params="leg_name parent pos_x pos_y pos_z roll pitch yaw fcp_joint_type:=prismatic">
     <!-- Base link -->
     <link name="${leg_name}_base_link">
@@ -7,5 +8,6 @@
         <origin xyz="-0.00979014713716649 -0.00139011782449186 0.0218935307853371" rpy="0 0 0" />
         <mass value="0.0808021222974834" />
-        <inertia ixx="1.27655E-05" ixy="5.10643E-13" ixz="-2.82428E-08" iyy="2.29991E-05" iyz="4.39699E-07" izz="1.62889E-05" />
+        <inertia ixx="1.27655E-05" ixy="5.10643E-13" ixz="-2.82428E-08" iyy="2.29991E-05"
+          iyz="4.39699E-07" izz="1.62889E-05" />
       </inertial>
       <visual>
@@ -14,5 +16,5 @@
           <mesh filename="package://elkapod_description/meshes/right_leg/base_link.STL" />
         </geometry>
-        <material name="leg_black"/>
+        <material name="leg_black" />
       </visual>
       <collision>
@@ -24,8 +26,8 @@
     </link>
     <joint name="${leg_name}_base_joint" type="fixed">
-        <origin xyz="${pos_x} ${pos_y} ${pos_z}" rpy="${roll} ${pitch} ${yaw}" />
-        <parent link="${parent}" />
-        <child link="${leg_name}_base_link" />
-        <axis xyz="0 0 0" />
+      <origin xyz="${pos_x} ${pos_y} ${pos_z}" rpy="${roll} ${pitch} ${yaw}" />
+      <parent link="${parent}" />
+      <child link="${leg_name}_base_link" />
+      <axis xyz="0 0 0" />
     </joint>
     <!-- Link A -->
@@ -34,5 +36,6 @@
         <origin xyz="0.0337988193565861 -0.000554586093327376 0.000549586085186449" rpy="0 0 0" />
         <mass value="0.0426933486153037" />
-        <inertia ixx="1.98022E-05" ixy="-2.13458E-13" ixz="-5.41372E-13" iyy="1.670609E-05" iyz="-2.17248E-12" izz="1.67061E-05" />
+        <inertia ixx="1.98022E-05" ixy="-2.13458E-13" ixz="-5.41372E-13" iyy="1.670609E-05"
+          iyz="-2.17248E-12" izz="1.67061E-05" />
       </inertial>
       <visual>
@@ -41,5 +44,5 @@
           <mesh filename="package://elkapod_description/meshes/right_leg/linkA.STL" />
         </geometry>
-        <material name="leg_black"/>
+        <material name="leg_black" />
       </visual>
       <collision>
@@ -52,9 +55,9 @@
     <!-- Joint J1 -->
     <joint name="${leg_name}_J1" type="revolute">
-        <origin xyz="0 0 0.02428" rpy="0 0 0" />
-        <parent link="${leg_name}_base_link" />
-        <child link="${leg_name}_linkA" />
-        <axis xyz="0 0 1" />
-        <limit lower="-1.57" upper="1.57" effort="50.0" velocity="7.3" />
+      <origin xyz="0 0 0.02428" rpy="0 0 0" />
+      <parent link="${leg_name}_base_link" />
+      <child link="${leg_name}_linkA" />
+      <axis xyz="0 0 1" />
+      <limit lower="-1.570796327" upper="1.570796327" effort="50.0" velocity="7.3" />
     </joint>
     <!-- Link B -->
@@ -63,5 +66,6 @@
         <origin xyz="0.0461949754482681 0.00470912944794107 -0.00261992673183065" rpy="0 0 0" />
         <mass value="0.168678406706635" />
-        <inertia ixx="2.79458E-05" ixy="8.13719E-13" ixz="2.16502E-12" iyy="4.53975E-05" iyz="-7.11437E-07" izz="3.38637E-05" />
+        <inertia ixx="2.79458E-05" ixy="8.13719E-13" ixz="2.16502E-12" iyy="4.53975E-05"
+          iyz="-7.11437E-07" izz="3.38637E-05" />
       </inertial>
       <visual>
@@ -70,5 +74,5 @@
           <mesh filename="package://elkapod_description/meshes/right_leg/linkB.STL" />
         </geometry>
-        <material name="leg_black"/>
+        <material name="leg_black" />
       </visual>
       <collision>
@@ -81,9 +85,9 @@
     <!-- Joint J2 -->
     <joint name="${leg_name}_J2" type="revolute">
-        <origin xyz="0.0676 0 0" rpy="1.5708 0 0" />
-        <parent link="${leg_name}_linkA" />
-        <child link="${leg_name}_linkB" />
-        <axis xyz="0 0 1" />
-        <limit lower="-1.57" upper="1.57" effort="50.0" velocity="7.3" />
+      <origin xyz="0.0676 0 0" rpy="1.570796327 0 0" />
+      <parent link="${leg_name}_linkA" />
+      <child link="${leg_name}_linkB" />
+      <axis xyz="0 0 1" />
+      <limit lower="-1.570796327" upper="1.570796327" effort="50.0" velocity="7.3" />
     </joint>
     <!-- Link C -->
@@ -92,5 +96,6 @@
         <origin xyz="0.0626878415018562 0.0138717503264788 0.00052553418423365" rpy="0 0 0" />
         <mass value="0.0457999682692435" />
-        <inertia ixx="1.77293E-05" ixy="-3.34917E-06" ixz="3.26962E-07" iyy="6.16756E-05" iyz="6.79304E-08" izz="5.23429E-05" />
+        <inertia ixx="1.77293E-05" ixy="-3.34917E-06" ixz="3.26962E-07" iyy="6.16756E-05"
+          iyz="6.79304E-08" izz="5.23429E-05" />
       </inertial>
       <visual>
@@ -99,5 +104,5 @@
           <mesh filename="package://elkapod_description/meshes/right_leg/linkC.STL" />
         </geometry>
-        <material name="orange_pla"/>
+        <material name="orange_pla" />
       </visual>
       <collision>
@@ -110,9 +115,9 @@
     <!-- Joint J3 -->
     <joint name="${leg_name}_J3" type="revolute">
-        <origin xyz="0.092358 -0.0014421 0" rpy="0 0 0" />
-        <parent link="${leg_name}_linkB" />
-        <child link="${leg_name}_linkC" />
-        <axis xyz="0 0 1" />
-        <limit lower="-3.14" upper="3.14" effort="50.0" velocity="7.3" />
+      <origin xyz="0.092358 -0.0014421 0" rpy="0 0 0" />
+      <parent link="${leg_name}_linkB" />
+      <child link="${leg_name}_linkC" />
+      <axis xyz="0 0 1" />
+      <limit lower="-3.141592654" upper="0.0" effort="50.0" velocity="7.3" />
     </joint>
     <!-- FCP link -->
@@ -121,10 +126,11 @@
         <origin xyz="0.000341547110338625 4.16333634234434E-17 -3.46944695195361E-17" rpy="0 0 0" />
         <mass value="0.0111617991818567" />
-        <inertia ixx="1.19862E-06" ixy="1.05879E-22" ixz="1.15499E-24" iyy="1.06703E-06" iyz="9.44775E-26" izz="1.06703E-06" />
+        <inertia ixx="1.19862E-06" ixy="1.05879E-22" ixz="1.15499E-24" iyy="1.06703E-06"
+          iyz="9.44775E-26" izz="1.06703E-06" />
       </inertial>
       <visual>
         <origin xyz="0 0 0" rpy="0 0 0" />
         <geometry>
-          <sphere radius="0.01"/>
+          <sphere radius="0.01" />
         </geometry>
         <material name="">
@@ -135,5 +141,5 @@
         <origin xyz="0 0 0" rpy="0 0 0" />
         <geometry>
-          <sphere radius="0.01"/>
+          <sphere radius="0.01" />
         </geometry>
       </collision>
@@ -146,18 +152,4 @@
       <minDepth>0.01</minDepth>
     </gazebo>
-    <!-- <gazebo reference="${leg_name}_FCP_joint">
-        <sensor name="${leg_name}_fsr" type="force_torque">
-          <always_on>true</always_on>
-          <update_rate>100</update_rate>
-          <visualize>true</visualize>
-          <topic>/legs/${leg_name}_fsr</topic>
-          <enable_metrics>true</enable_metrics>
-          <pose>0 0 0 0 0 0</pose>
-          <force_torque>
-            <frame>sensor</frame>
-            <measure_direction>child_to_parent</measure_direction>
-          </force_torque>
-        </sensor>
-    </gazebo> -->
     <gazebo reference="${leg_name}_FCP">
       <sensor name="contact" type="contact">
@@ -171,11 +163,11 @@
     </gazebo>
     <!-- Fixed joint for FCP -->
-    <joint name="${leg_name}_FCP_joint" type="prismatic">
-        <origin xyz="0.213503787197785 0.00857470533092818 0" rpy="0 0 -0.294032099334707" />
-        <parent link="${leg_name}_linkC" />
-        <child link="${leg_name}_FCP" />
-        <axis xyz="1 0 0" />
-        <limit effort="1000.0" lower="-0.0001" upper="0.0001" velocity="30"/>
-        <dynamics damping="10.0" friction="0.0"/>
+    <joint name="${leg_name}_FCP_joint" type="${fcp_joint_type}">
+      <origin xyz="0.213503787197785 0.00857470533092818 0" rpy="0 0 -0.294032099334707" />
+      <parent link="${leg_name}_linkC" />
+      <child link="${leg_name}_FCP" />
+      <axis xyz="1 0 0" />
+      <limit effort="1000.0" lower="-0.0001" upper="0.0001" velocity="30" />
+      <dynamics damping="10.0" friction="0.0" />
     </joint>
   </xacro:macro>

File: elkapod_description/urdf/sensors/depth_camera.xacro (robot description, xacro)
@@ -35,5 +35,5 @@
         <axis xyz="0 0 0" />
     </joint>
-    <xacro:macro name="elkapod_sensors_fron_camera" params="sim_mode:=^|false">
+    <xacro:macro name="elkapod_sensors_front_camera" params="sim_mode:=^|false">
         <xacro:if value="${sim_mode}">
             <gazebo reference="front_camera_optical">
